File: DRV8711.sch (EAGLE design)
At the start: 37 parts, among them IC1 DRV8711, T1 IPC50N04S5, T2 IPC50N04S5, T3 IPC50N04S5, T4 IPC50N04S5, T5 IPC50N04S5, T6 IPC50N04S5, T7 IPC50N04S5, T8 IPC50N04S5

Commit message: Add files via upload
Parts:
- removed JP2: (no value), pinhead:PINHD-1X3
- added R17, R18, R19: 0R, rcl:R-EU_R0805
- added STALL/BEMF: (no value), pinhead:PINHD-1X3
Connections:
- net +5V: now also STALL/BEMF.1; no longer JP2.1
- net AGND: now also R17.1, R18.1, R19.1, X2-1.KL
- net FAULT: now also STALL/BEMF.3; no longer JP2.3
- net GND: now also R17.2, R18.2, R19.2; no longer X2-1.KL
- net STALL: now also STALL/BEMF.2; no longer JP2.2
Other:
- moved on the sheet: C1, C2, C3, C4, C5, C6, C7, COM, CONTROL, IC1, R15, R16

Commit message: Add files via upload
without 5 parallel resistors
Parts:
- removed R10, R11, R3, R4, R5, R7, R8, R9: (no value), rcl:R-EU_R0805
- removed R19: 0R, rcl:R-EU_R0805
- added C8: 1mF, SparkFun-Capacitors:1000UF-RADIAL-5MM-25V-20%
- R1, R2: value (none) -> 0.05R/5W; device rcl:R-EU_R0805 -> rcl:R-EU_R4527
Connections:
- net AGND: no longer R10.1, R11.1, R19.1, R3.1, R4.1, R5.1, R7.1, R8.1, R9.1
- net AISENP: no longer R2.2, R3.2, R4.2, R5.2
- net AOUT1: now also X1-1.KL; no longer X1-4.KL
- net AOUT2: now also X1-2.KL; no longer X1-3.KL
- net BISENP: now also R2.2; no longer R10.2, R11.2, R7.2, R8.2, R9.2
- net BOUT1: now also X1-3.KL; no longer X1-2.KL
- net BOUT2: now also X1-4.KL; no longer X1-1.KL
- net FAULT: now also STALL/BEMF.2; no longer STALL/BEMF.3
- net GND: now also C8.-; no longer R19.2
- net STALL: now also STALL/BEMF.3; no longer STALL/BEMF.2
- net V+: now also C8.+
Other:
- moved on the sheet: R1, R2

Commit message: Add files via upload
Parts:
- R1, R2: value 0.05R/5W -> 0.3R/2W; device rcl:R-EU_R4527 -> rcl:R-EU_R2512
Changed lines of the file:
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@@
 <part name="AGND1" library="supply1" library_urn="urn:adsk.eagle:library:371" deviceset="AGND" device=""/>
 <part name="GND6" library="SparkFun-PowerSymbols" library_urn="urn:adsk.eagle:library:530" deviceset="GND" device=""/>
-<part name="R1" library="rcl" library_urn="urn:adsk.eagle:library:334" deviceset="R-EU_" device="R4527" package3d_urn="urn:adsk.eagle:package:13310/2" value="0.05R/5W"/>
-<part name="R2" library="rcl" library_urn="urn:adsk.eagle:library:334" deviceset="R-EU_" device="R4527" package3d_urn="urn:adsk.eagle:package:13310/2" value="0.05R/5W"/>
 <part name="C8" library="SparkFun-Capacitors" library_urn="urn:adsk.eagle:library:510" deviceset="1000UF" device="-RADIAL-5MM-25V-20%" package3d_urn="urn:adsk.eagle:package:37412/1" value="1mF"/>
 <part name="SUPPLY5" library="supply2" library_urn="urn:adsk.eagle:library:372" deviceset="V+" device=""/>
 <part name="GND7" library="SparkFun-PowerSymbols" library_urn="urn:adsk.eagle:library:530" deviceset="GND" device=""/>
+<part name="R1" library="rcl" library_urn="urn:adsk.eagle:library:334" deviceset="R-EU_" device="R2512" package3d_urn="urn:adsk.eagle:package:23545/2" value="0.3R/2W"/>
+<part name="R2" library="rcl" library_urn="urn:adsk.eagle:library:334" deviceset="R-EU_" device="R2512" package3d_urn="urn:adsk.eagle:package:23545/2" value="0.3R/2W"/>
 </parts>
 <sheets>
@@
 <attribute name="VALUE" x="180.34" y="88.646" size="1.778" layer="96" align="top-center"/>
 </instance>
-<instance part="R1" gate="G$1" x="127" y="121.92" smashed="yes" rot="R90">
-<attribute name="NAME" x="123.19" y="125.5014" size="1.778" layer="95" rot="R180"/>
-<attribute name="VALUE" x="123.19" y="122.682" size="1.778" layer="96" rot="R180"/>
-</instance>
-<instance part="R2" gate="G$1" x="205.74" y="121.92" smashed="yes" rot="R90">
-<attribute name="NAME" x="201.93" y="125.5014" size="1.778" layer="95" rot="R180"/>
-<attribute name="VALUE" x="201.93" y="122.682" size="1.778" layer="96" rot="R180"/>
-</instance>
 <instance part="C8" gate="G$1" x="241.3" y="71.12" smashed="yes">
 <attribute name="NAME" x="242.316" y="71.755" size="1.778" layer="95" font="vector"/>
@@
 <instance part="GND7" gate="1" x="241.3" y="58.42" smashed="yes">
 <attribute name="VALUE" x="241.3" y="58.166" size="1.778" layer="96" align="top-center"/>
+</instance>
+<instance part="R1" gate="G$1" x="127" y="121.92" smashed="yes" rot="R90">
+<attribute name="NAME" x="125.73" y="125.5014" size="1.778" layer="95" rot="R180"/>
+<attribute name="VALUE" x="125.73" y="120.142" size="1.778" layer="96" rot="R180"/>
+</instance>
+<instance part="R2" gate="G$1" x="205.74" y="121.92" smashed="yes" rot="R90">
+<attribute name="NAME" x="204.47" y="125.5014" size="1.778" layer="95" rot="R180"/>
+<attribute name="VALUE" x="204.47" y="120.142" size="1.778" layer="96" rot="R180"/>
 </instance>
 </instances>
@@
 <wire x1="119.38" y1="129.54" x2="104.14" y2="129.54" width="0.1524" layer="91"/>
 <label x="106.68" y="129.54" size="1.778" layer="95"/>
-<pinref part="R1" gate="G$1" pin="2"/>
 <wire x1="127" y1="127" x2="127" y2="129.54" width="0.1524" layer="91"/>
 <junction x="127" y="129.54"/>
+<pinref part="R1" gate="G$1" pin="2"/>
 </segment>
 <segment>
@@
 <segment>
 <label x="106.68" y="114.3" size="1.778" layer="95"/>
-<pinref part="R1" gate="G$1" pin="1"/>
 <wire x1="127" y1="114.3" x2="104.14" y2="114.3" width="0.1524" layer="91"/>
 <wire x1="127" y1="116.84" x2="127" y2="114.3" width="0.1524" layer="91"/>
+<pinref part="R1" gate="G$1" pin="1"/>
 </segment>
 <segment>
 <label x="185.42" y="114.3" size="1.778" layer="95"/>
-<pinref part="R2" gate="G$1" pin="1"/>
 <wire x1="205.74" y1="114.3" x2="182.88" y2="114.3" width="0.1524" layer="91"/>
 <wire x1="205.74" y1="116.84" x2="205.74" y2="114.3" width="0.1524" layer="91"/>
+<pinref part="R2" gate="G$1" pin="1"/>
 </segment>
 <segment>
@@
 <wire x1="198.12" y1="129.54" x2="182.88" y2="129.54" width="0.1524" layer="91"/>
 <label x="185.42" y="129.54" size="1.778" layer="95"/>
-<pinref part="R2" gate="G$1" pin="2"/>
 <wire x1="205.74" y1="127" x2="205.74" y2="129.54" width="0.1524" layer="91"/>
 <junction x="205.74" y="129.54"/>
-</segment>
-<segment>
+<pinref part="R2" gate="G$1" pin="2"/>
+</segment>
+<segment>
